File: cociclo_05/hardware/cociclo_05.sch (EAGLE design)
At the start: 9 parts, among them J1 PMS7003

Commit message: hasta la 1.0 :)
Adición logo unloquer
Adición opción para Adafruit MAX 4466
Adición ‘screw terminal’
Parts:
- added MAX4466ADAFRUIT: (no value), SparkFun-Connectors:M03PTH
- added SCREWTERMINAL: (no value), SparkFun-Connectors:M023.5MM
- renumbered LED to SK9822LED
Connections:
- net +5V: now also SCREWTERMINAL.1
- net 10SET: no longer JP1.7
- net CH_PD: now also MAX4466ADAFRUIT.3
- net GND: now also MAX4466ADAFRUIT.2, SCREWTERMINAL.2
- net MQ7ANALOG: now also MAX4466ADAFRUIT.1
Changed lines of the file:
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@@
 <part name="JP1" library="SparkFun-Connectors" deviceset="M08" device=""/>
 <part name="JP2" library="SparkFun-Connectors" deviceset="M08" device=""/>
-<part name="LED" library="jos-ph" deviceset="APA102" device="5050"/>
+<part name="SK9822LED" library="jos-ph" deviceset="APA102" device="5050"/>
 <part name="J1" library="Board-to-Board (rev18a)" deviceset="621X1021021" device="" value="PMS7003"/>
+<part name="MAX4466ADAFRUIT" library="SparkFun-Connectors" library_urn="urn:adsk.eagle:library:6242394" deviceset="M03" device="PTH" package3d_urn="urn:adsk.eagle:package:6242963/1"/>
+<part name="SCREWTERMINAL" library="SparkFun-Connectors" library_urn="urn:adsk.eagle:library:6242394" deviceset="M02" device="3.5MM" package3d_urn="urn:adsk.eagle:package:6242944/1"/>
 </parts>
 <sheets>
@@
 <instance part="JP1" gate="G$1" x="45.72" y="55.88" rot="R180"/>
 <instance part="JP2" gate="G$1" x="58.42" y="53.34"/>
-<instance part="LED" gate="G$1" x="86.36" y="88.9"/>
+<instance part="SK9822LED" gate="G$1" x="86.36" y="88.9"/>
 <instance part="J1" gate="G$1" x="111.76" y="38.1" rot="R90"/>
+<instance part="MAX4466ADAFRUIT" gate="G$1" x="68.58" y="17.78"/>
+<instance part="SCREWTERMINAL" gate="G$1" x="106.68" y="15.24" rot="MR0"/>
 </instances>
 <busses>
@@
 <pinref part="R1" gate="G$1" pin="1"/>
 <wire x1="81.28" y1="40.64" x2="83.82" y2="40.64" width="0.1524" layer="91"/>
-<wire x1="63.5" y1="48.26" x2="83.82" y2="48.26" width="0.1524" layer="91"/>
+<wire x1="63.5" y1="48.26" x2="81.28" y2="48.26" width="0.1524" layer="91"/>
 <pinref part="DHT11" gate="G$1" pin="4"/>
+<wire x1="81.28" y1="48.26" x2="83.82" y2="48.26" width="0.1524" layer="91"/>
 <wire x1="25.4" y1="78.74" x2="83.82" y2="78.74" width="0.1524" layer="91"/>
-<pinref part="LED" gate="G$1" pin="GND"/>
+<pinref part="SK9822LED" gate="G$1" pin="GND"/>
 <wire x1="83.82" y1="83.82" x2="83.82" y2="78.74" width="0.1524" layer="91"/>
 <wire x1="83.82" y1="78.74" x2="83.82" y2="48.26" width="0.1524" layer="91"/>
-<wire x1="83.82" y1="48.26" x2="109.22" y2="48.26" width="0.1524" layer="91"/>
+<wire x1="83.82" y1="48.26" x2="91.44" y2="48.26" width="0.1524" layer="91"/>
+<wire x1="91.44" y1="48.26" x2="109.22" y2="48.26" width="0.1524" layer="91"/>
 <wire x1="109.22" y1="45.72" x2="109.22" y2="48.26" width="0.1524" layer="91"/>
 <pinref part="J1" gate="G$1" pin="9"/>
 <pinref part="J1" gate="G$1" pin="2"/>
 <wire x1="109.22" y1="45.72" x2="109.22" y2="30.48" width="0.1524" layer="91"/>
+<pinref part="MAX4466ADAFRUIT" gate="G$1" pin="2"/>
+<wire x1="76.2" y1="17.78" x2="81.28" y2="17.78" width="0.1524" layer="91"/>
+<wire x1="81.28" y1="17.78" x2="81.28" y2="48.26" width="0.1524" layer="91"/>
+<wire x1="91.44" y1="48.26" x2="91.44" y2="17.78" width="0.1524" layer="91"/>
+<wire x1="91.44" y1="17.78" x2="99.06" y2="17.78" width="0.1524" layer="91"/>
+<pinref part="SCREWTERMINAL" gate="G$1" pin="2"/>
+<wire x1="99.06" y1="17.78" x2="104.14" y2="17.78" width="0.1524" layer="91"/>
+<junction x="99.06" y="17.78"/>
 </segment>
 </net>
@@
 <pinref part="JP1" gate="G$1" pin="8"/>
 <wire x1="30.48" y1="66.04" x2="40.64" y2="45.72" width="0.1524" layer="91"/>
+<pinref part="MAX4466ADAFRUIT" gate="G$1" pin="3"/>
 <wire x1="40.64" y1="45.72" x2="45.72" y2="45.72" width="0.1524" layer="91"/>
+<wire x1="76.2" y1="20.32" x2="76.2" y2="25.4" width="0.1524" layer="91"/>
+<wire x1="76.2" y1="25.4" x2="60.96" y2="25.4" width="0.1524" layer="91"/>
+<wire x1="60.96" y1="25.4" x2="60.96" y2="10.16" width="0.1524" layer="91"/>
+<wire x1="60.96" y1="10.16" x2="38.1" y2="10.16" width="0.1524" layer="91"/>
+<wire x1="38.1" y1="10.16" x2="38.1" y2="45.72" width="0.1524" layer="91"/>
+<wire x1="38.1" y1="45.72" x2="40.64" y2="45.72" width="0.1524" layer="91"/>
 </segment>
 </net>
@@
 <wire x1="63.5" y1="45.72" x2="55.88" y2="22.86" width="0.1524" layer="91"/>
 <pinref part="JP2" gate="G$1" pin="1"/>
-<wire x1="99.06" y1="45.72" x2="63.5" y2="45.72" width="0.1524" layer="91"/>
+<wire x1="99.06" y1="45.72" x2="93.98" y2="45.72" width="0.1524" layer="91"/>
+<wire x1="93.98" y1="45.72" x2="63.5" y2="45.72" width="0.1524" layer="91"/>
 <wire x1="63.5" y1="45.72" x2="58.42" y2="45.72" width="0.1524" layer="91"/>
 <wire x1="99.06" y1="45.72" x2="99.06" y2="99.06" width="0.1524" layer="91"/>
-<pinref part="LED" gate="G$1" pin="VCC"/>
+<pinref part="SK9822LED" gate="G$1" pin="VCC"/>
 <wire x1="99.06" y1="99.06" x2="86.36" y2="99.06" width="0.1524" layer="91"/>
 <pinref part="J1" gate="G$1" pin="10"/>
@@
 <pinref part="J1" gate="G$1" pin="1"/>
 <wire x1="106.68" y1="45.72" x2="106.68" y2="30.48" width="0.1524" layer="91"/>
+<wire x1="93.98" y1="45.72" x2="93.98" y2="27.94" width="0.1524" layer="91"/>
+<pinref part="SCREWTERMINAL" gate="G$1" pin="1"/>
+<wire x1="93.98" y1="27.94" x2="99.06" y2="15.24" width="0.1524" layer="91"/>
 </segment>
 </net>
@@
 <pinref part="MQ-7" gate="G$1" pin="1"/>
 <wire x1="55.88" y1="30.48" x2="71.12" y2="30.48" width="0.1524" layer="91"/>
+<wire x1="76.2" y1="30.48" x2="71.12" y2="30.48" width="0.1524" layer="91"/>
+<pinref part="MAX4466ADAFRUIT" gate="G$1" pin="1"/>
+<wire x1="76.2" y1="15.24" x2="78.74" y2="15.24" width="0.1524" layer="91"/>
+<wire x1="78.74" y1="15.24" x2="78.74" y2="30.48" width="0.1524" layer="91"/>
+<wire x1="78.74" y1="30.48" x2="71.12" y2="30.48" width="0.1524" layer="91"/>
 </segment>
 </net>
@@
 <wire x1="63.5" y1="55.88" x2="68.58" y2="55.88" width="0.1524" layer="91"/>
 <wire x1="68.58" y1="55.88" x2="68.58" y2="93.98" width="0.1524" layer="91"/>
-<pinref part="LED" gate="G$1" pin="DI"/>
+<pinref part="SK9822LED" gate="G$1" pin="DI"/>
 <wire x1="73.66" y1="93.98" x2="68.58" y2="93.98" width="0.1524" layer="91"/>
 </segment>
@@
 <wire x1="71.12" y1="53.34" x2="71.12" y2="88.9" width="0.1524" layer="91"/>
 <wire x1="71.12" y1="88.9" x2="73.66" y2="88.9" width="0.1524" layer="91"/>
-<pinref part="LED" gate="G$1" pin="CI"/>
+<pinref part="SK9822LED" gate="G$1" pin="CI"/>
 <wire x1="73.66" y1="88.9" x2="76.2" y2="88.9" width="0.1524" layer="91"/>
 <junction x="73.66" y="88.9"/>
@@
 <segment>
 <wire x1="116.84" y1="33.02" x2="116.84" y2="30.48" width="0.1524" layer="91"/>
-<wire x1="116.84" y1="30.48" x2="116.84" y2="15.24" width="0.1524" layer="91"/>
-<wire x1="116.84" y1="15.24" x2="30.48" y2="15.24" width="0.1524" layer="91"/>
-<wire x1="30.48" y1="15.24" x2="30.48" y2="48.26" width="0.1524" layer="91"/>
 <pinref part="J1" gate="G$1" pin="5"/>
-<junction x="116.84" y="30.48"/>
-<pinref part="JP1" gate="G$1" pin="7"/>
-<wire x1="40.64" y1="48.26" x2="30.48" y2="48.26" width="0.1524" layer="91"/>
 </segment>
 </net>
@@
 </schematic>
 </drawing>
+<compatibility>
+<note version="8.2" severity="warning">
+Since Version 8.2, EAGLE supports online libraries. The ids
+of those online libraries will not be understood (or retained)
+with this version.
+</note>
+<note version="8.3" severity="warning">
+Since Version 8.3, EAGLE supports URNs for individual library
+assets (packages, symbols, and devices). The URNs of those assets
+will not be understood (or retained) with this version.
+</note>
+<note version="8.3" severity="warning">
+Since Version 8.3, EAGLE supports the association of 3D packages
+with devices in libraries, schematics, and board files. Those 3D
+packages will not be understood (or retained) with this version.
+</note>
+</compatibility>
 </eagle>
